File: Poseidon/Poseidon.sch (EAGLE design)
At the start: 31 parts, among them Q1 2N5089, Q2 2N3906, Q3 2N5089, SW1 3PDT

Commit message: New board for Poseidon
Parts:
- removed C6: 100uF, caps-elec:0631
- removed D4: 1N4148, diodes:DO35.3
- removed DC: BATTERYBAT2, jacks:BATTERYBAT2
- removed GND: GND_PADROUND, supply pins:GND_PADROUND
- added C1: 47n, caps-film:CAP.2
- added D1: 1N4001, diodes:DO41.3
- added PWR: PJ-037A, PJ-037A:PJ-037A
- C3: value 47n -> 100uF; device caps-film:CAP.2 -> caps-elec:0631
- D3: value 1N4001 -> 1N4148; device diodes:DO41.3 -> diodes:DO35.3
- IN: value IN -> NV-PJ3410_MONO; device supply pins:IN -> MusicThingModular:NV-PJ3410_MONO
- OUT: value OUT -> NV-PJ3410_MONO; device supply pins:OUT -> MusicThingModular:NV-PJ3410_MONO
- R1: value 2.2M -> 68k
- R10: value 22k -> 10k
- R11: value 22k -> 6.2k
- R12: value 10k -> 560k
- R13: value 47k -> 160k
- R14: value 4.7k -> 2.2M
- R2: value 160k -> 68k
- R3: value 560k -> 22k
- R4: value 18k -> 22k
- R6: value 6.2k -> 47k
- R7: value 10k -> 4.7k
- R8: value 68k -> 10k
- R9: value 68k -> 18k
- renumbered SW1 to 3PDT
Connections:
- removed net IN: 3PDTA.2, IN.IN
- removed net OUT: 3PDTB.2, OUT.OUT
- new net N$13: 3PDTB.2, OUT.TIP
- new net N$8: 3PDTA.2, IN.TIP
- net +9V: now also C3.+, D1.C, PWR.1, R10.2, R12.2, R7.2, R9.2; no longer C6.+, D3.C, DC.P$1, R11.2, R14.2, R4.2, R5.2
- net CIN: now also C5.1, R14.2; no longer C2.1, R1.2
- net COUT: now also C2.2, R6.2; no longer C5.2, R13.2
- net GND: now also 3PDTC.3, C3.-, D1.A, IN.SLEEVE, IN.SWITCH, OUT.SLEEVE, OUT.SWITCH, PWR.2, R11.1, R14.1, R4.1, R5.1, R8.1; no longer C6.-, D3.A, DC.P$2, GND.GND, R1.1, R10.1, R12.1, R2.1, R7.1
- net N$10: now also D2.A, R1.1; no longer D4.A, R9.1
- net N$11: now also R1.2, R2.1, R3.1, R4.2; no longer R10.2, R11.1, R8.1, R9.2
- net N$12: now also C1.2, D3.A, R2.2; no longer C3.2, D2.A, R8.2
- net N$14: now also D3.C; no longer D4.C
- net N$16: now also C2.1, R5.2; no longer C5.1, R12.2
- net N$2: now also C5.2, R12.1, R13.2; no longer C2.2, R2.2, R3.1
- net N$4: now also R11.2; no longer R6.2
- net N$5: now also R7.1; no longer R14.1
- net N$6: now also R9.1; no longer R4.1
- net N$7: now also C1.1, R10.1; no longer C3.1, R5.1
- net N$9: now also R8.2; no longer R7.2
Other:
- moved on the sheet: C2, C5, D2, D3, LED, R1, R10, R11, R12, R13, R14, R2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
