File: Poseidon/Poseidon.brd (EAGLE design)
At the start: 38 x 84 mm, 30 parts, among them Q1 2N5089, Q2 2N3906, Q3 2N5089

Commit message: Added boards
Other:
- outline, holes or cut-outs redrawn
- board text added: "REV 0.0"
Changed lines of the file:
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@@
 <wire x1="37" y1="83" x2="1" y2="83" width="0.254" layer="42"/>
 <wire x1="1" y1="83" x2="1" y2="71" width="0.254" layer="42"/>
-<wire x1="0" y1="0" x2="38" y2="0" width="0" layer="20"/>
-<wire x1="38" y1="0" x2="38" y2="84" width="0" layer="20"/>
-<wire x1="38" y1="84" x2="0" y2="84" width="0" layer="20"/>
-<wire x1="0" y1="84" x2="0" y2="0" width="0" layer="20"/>
 <rectangle x1="36.605009375" y1="7.828034375" x2="36.815828125" y2="7.870196875" layer="25" rot="R90"/>
 <rectangle x1="36.32941875" y1="9.28980625" x2="37.09141875" y2="9.33196875" layer="25" rot="R90"/>
@@
 <rectangle x1="3.176728125" y1="16.653334375" x2="4.192728125" y2="16.695753125" layer="25" rot="R90"/>
 <rectangle x1="3.51581875" y1="18.05160625" x2="3.8536375" y2="18.094025" layer="25" rot="R90"/>
+<wire x1="0" y1="81" x2="3" y2="84" width="0" layer="20" curve="-90"/>
+<wire x1="3" y1="84" x2="35" y2="84" width="0" layer="20"/>
+<wire x1="35" y1="84" x2="38" y2="81" width="0" layer="20" curve="-90"/>
+<wire x1="38" y1="81" x2="38" y2="3" width="0" layer="20"/>
+<wire x1="38" y1="3" x2="35" y2="0" width="0" layer="20" curve="-90"/>
+<wire x1="35" y1="0" x2="3" y2="0" width="0" layer="20"/>
+<wire x1="3" y1="0" x2="0" y2="3" width="0" layer="20" curve="-90"/>
+<wire x1="0" y1="3" x2="0" y2="81" width="0" layer="20"/>
+<text x="16" y="21" size="1.016" layer="21">REV 0.0</text>
 </plain>
 <attributes>
@@
 </element>
 <element name="3PDT" library="switches" package="3PDT" value="3PDT" x="19" y="12" smashed="yes" rot="MR0">
-<attribute name="NAME" x="15.805" y="18.82" size="1.27" layer="21" ratio="12"/>
+<attribute name="NAME" x="16.605" y="19.22" size="1.27" layer="21" ratio="12"/>
 </element>
 <element name="IN" library="MusicThingModular" package="NV-PJ3410_SOCKET_MONO" value="NV-PJ3410_MONO" x="7" y="75" smashed="yes" rot="MR0">
