File: 3PDT_Breakout/3PDT_Breakout.sch (EAGLE design)
At the start: 12 parts

Commit message: Added boards
Parts:
- removed CI, CO: PADS.SQR_NL, supply pins:PADS.SQR_NL
- removed GI, GND, GO: GND_PADROUND, supply pins:GND_PADROUND
- removed I: IN, supply pins:IN
- removed LED: LED3MM, diodes:LED3MM
- removed O: OUT, supply pins:OUT
- removed V+: +9V_PAD, supply pins:+9V_PAD
- added U$1: HEADERS8, my_headers:HEADERS8
Connections:
- removed net N$3: 3PDTB.1, CO.P$1
- removed net N$4: 3PDTA.1, CI.P$1
- new net CI: 3PDTB.1, U$1.CI
- new net CO: 3PDTA.1, U$1.CO
- net +9V: now also U$1.+9V; no longer V+.+9V
- net GND: now also U$1.G1, U$1.G2, U$1.GND; no longer GI.GND, GND.GND, GO.GND
- net IN: now also 3PDTB.2, U$1.IN; no longer 3PDTA.2, I.IN
- net N$1: no longer LED.C
- net N$2: no longer LED.A
- net OUT: now also 3PDTA.2, U$1.OUT; no longer 3PDTB.2, O.OUT
Other:
- moved on the sheet: LED1
Changed lines of the file:
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@@
 <parts>
 <part name="3PDT" library="switches" deviceset="3PDT" device=""/>
-<part name="I" library="supply pins" deviceset="IN" device=""/>
-<part name="O" library="supply pins" deviceset="OUT" device=""/>
 <part name="CLR" library="resistors" deviceset="RESISTORS" device=".3B"/>
-<part name="LED" library="diodes" deviceset="LED" device="3MM"/>
 <part name="LED1" library="diodes" deviceset="LED" device="3MM"/>
 <part name="GND1" library="supply pins" deviceset="GND" device=""/>
 <part name="V1" library="supply pins" deviceset="+9V" device=""/>
-<part name="GO" library="supply pins" deviceset="GND_PAD" device="ROUND"/>
-<part name="GI" library="supply pins" deviceset="GND_PAD" device="ROUND"/>
-<part name="CO" library="supply pins" deviceset="PADS." device="SQR_NL"/>
-<part name="CI" library="supply pins" deviceset="PADS." device="SQR_NL"/>
-<part name="V+" library="supply pins" deviceset="+9V_PAD" device=""/>
-<part name="GND" library="supply pins" deviceset="GND_PAD" device="ROUND"/>
+<part name="U$1" library="my_headers" deviceset="HEADERS8" device=""/>
 </parts>
 <sheets>
@@
 <attribute name="NAME" x="43.053" y="47.625" size="1.778" layer="95"/>
 </instance>
-<instance part="I" gate="G$1" x="38.1" y="68.58" smashed="yes">
-<attribute name="NAME" x="38.1" y="73.66" size="1.778" layer="95" rot="R180"/>
-</instance>
-<instance part="O" gate="G$1" x="38.1" y="55.88" smashed="yes" rot="R180">
-<attribute name="NAME" x="38.1" y="53.34" size="1.778" layer="95" rot="R180"/>
-</instance>
 <instance part="CLR" gate="G$1" x="83.82" y="45.72" smashed="yes">
 <attribute name="NAME" x="82.169" y="47.2186" size="1.778" layer="95"/>
 <attribute name="VALUE" x="81.407" y="42.672" size="1.778" layer="96"/>
 </instance>
-<instance part="LED" gate="G$1" x="66.04" y="45.72" smashed="yes">
+<instance part="LED1" gate="G$1" x="66.04" y="45.72" smashed="yes">
 <attribute name="NAME" x="64.008" y="42.164" size="1.778" layer="95"/>
-</instance>
-<instance part="LED1" gate="G$1" x="66.04" y="38.1" smashed="yes">
-<attribute name="NAME" x="64.008" y="34.544" size="1.778" layer="95"/>
 </instance>
 <instance part="GND1" gate="GND" x="35.56" y="17.78" smashed="yes">
@@
 <attribute name="VALUE" x="93.345" y="14.605" size="1.778" layer="96" rot="R180"/>
 </instance>
-<instance part="GO" gate="GND" x="40.64" y="17.78" smashed="yes">
-<attribute name="VALUE" x="38.735" y="14.605" size="1.778" layer="96"/>
-</instance>
-<instance part="GI" gate="GND" x="45.72" y="17.78" smashed="yes">
-<attribute name="VALUE" x="43.815" y="14.605" size="1.778" layer="96"/>
-</instance>
-<instance part="CO" gate="G$1" x="60.96" y="58.42" smashed="yes" rot="R270"/>
-<instance part="CI" gate="G$1" x="60.96" y="71.12" smashed="yes" rot="R270"/>
-<instance part="V+" gate="+9V" x="68.58" y="22.86" smashed="yes">
-<attribute name="VALUE" x="66.675" y="26.035" size="1.778" layer="96"/>
-</instance>
-<instance part="GND" gate="GND" x="53.34" y="22.86" smashed="yes" rot="R180">
-<attribute name="VALUE" x="55.245" y="26.035" size="1.778" layer="96" rot="R180"/>
-</instance>
+<instance part="U$1" gate="G$1" x="15.24" y="45.72" smashed="yes" rot="R180"/>
 </instances>
 <busses>
@@
 <segment>
 <pinref part="3PDT" gate="C" pin="1"/>
-<pinref part="LED" gate="G$1" pin="C"/>
-<wire x1="55.88" y1="45.72" x2="60.96" y2="45.72" width="0.1524" layer="91"/>
+<wire x1="55.88" y1="45.72" x2="63.5" y2="45.72" width="0.1524" layer="91"/>
 <pinref part="LED1" gate="G$1" pin="C"/>
-<wire x1="60.96" y1="45.72" x2="63.5" y2="45.72" width="0.1524" layer="91"/>
-<wire x1="60.96" y1="45.72" x2="60.96" y2="38.1" width="0.1524" layer="91"/>
-<wire x1="60.96" y1="38.1" x2="63.5" y2="38.1" width="0.1524" layer="91"/>
-<junction x="60.96" y="45.72"/>
 </segment>
 </net>
 <net name="N$2" class="0">
 <segment>
-<pinref part="LED" gate="G$1" pin="A"/>
 <pinref part="CLR" gate="G$1" pin="1"/>
-<wire x1="71.12" y1="45.72" x2="73.66" y2="45.72" width="0.1524" layer="91"/>
 <pinref part="LED1" gate="G$1" pin="A"/>
-<wire x1="73.66" y1="45.72" x2="78.74" y2="45.72" width="0.1524" layer="91"/>
-<wire x1="71.12" y1="38.1" x2="73.66" y2="38.1" width="0.1524" layer="91"/>
-<wire x1="73.66" y1="38.1" x2="73.66" y2="45.72" width="0.1524" layer="91"/>
-<junction x="73.66" y="45.72"/>
+<wire x1="71.12" y1="45.72" x2="78.74" y2="45.72" width="0.1524" layer="91"/>
 </segment>
 </net>
@@
 <pinref part="3PDT" gate="C" pin="3"/>
 <wire x1="58.42" y1="40.64" x2="55.88" y2="40.64" width="0.1524" layer="91"/>
-<wire x1="53.34" y1="20.32" x2="45.72" y2="20.32" width="0.1524" layer="91"/>
-<wire x1="45.72" y1="20.32" x2="40.64" y2="20.32" width="0.1524" layer="91"/>
-<wire x1="40.64" y1="20.32" x2="35.56" y2="20.32" width="0.1524" layer="91"/>
 <wire x1="35.56" y1="20.32" x2="35.56" y2="43.18" width="0.1524" layer="91"/>
 <pinref part="GND1" gate="GND" pin="GND"/>
-<junction x="35.56" y="20.32"/>
-<pinref part="GO" gate="GND" pin="GND"/>
-<junction x="40.64" y="20.32"/>
-<pinref part="GI" gate="GND" pin="GND"/>
-<junction x="45.72" y="20.32"/>
-<pinref part="GND" gate="GND" pin="GND"/>
+<label x="35.56" y="43.18" size="1.778" layer="95" rot="R180" xref="yes"/>
+</segment>
+<segment>
+<pinref part="U$1" gate="G$1" pin="G1"/>
+<junction x="12.7" y="27.94"/>
+<label x="15.24" y="27.94" size="1.778" layer="95"/>
+</segment>
+<segment>
+<pinref part="U$1" gate="G$1" pin="GND"/>
+<junction x="12.7" y="38.1"/>
+<label x="15.24" y="38.1" size="1.778" layer="95"/>
+</segment>
+<segment>
+<pinref part="U$1" gate="G$1" pin="G2"/>
+<junction x="12.7" y="45.72"/>
+<label x="15.24" y="45.72" size="1.778" layer="95"/>
 </segment>
 </net>
@@
 <pinref part="CLR" gate="G$1" pin="2"/>
 <wire x1="88.9" y1="45.72" x2="91.44" y2="45.72" width="0.1524" layer="91"/>
-<wire x1="68.58" y1="20.32" x2="91.44" y2="20.32" width="0.1524" layer="91"/>
 <wire x1="91.44" y1="20.32" x2="91.44" y2="45.72" width="0.1524" layer="91"/>
 <pinref part="V1" gate="+9V" pin="+9V"/>
-<junction x="91.44" y="20.32"/>
-<pinref part="V+" gate="+9V" pin="+9V"/>
+<label x="91.44" y="45.72" size="1.778" layer="95" xref="yes"/>
+</segment>
+<segment>
+<pinref part="U$1" gate="G$1" pin="+9V"/>
+<junction x="12.7" y="35.56"/>
+<label x="15.24" y="35.56" size="1.778" layer="95"/>
 </segment>
 </net>
 <net name="IN" class="0">
 <segment>
-<pinref part="I" gate="G$1" pin="IN"/>
-<pinref part="3PDT" gate="A" pin="2"/>
-<wire x1="40.64" y1="68.58" x2="45.72" y2="68.58" width="0.1524" layer="91"/>
+<pinref part="U$1" gate="G$1" pin="IN"/>
+<junction x="12.7" y="30.48"/>
+<label x="15.24" y="30.48" size="1.778" layer="95"/>
+</segment>
+<segment>
+<pinref part="3PDT" gate="B" pin="2"/>
+<junction x="45.72" y="55.88"/>
+<label x="45.72" y="55.88" size="1.778" layer="95" rot="R180"/>
 </segment>
 </net>
 <net name="OUT" class="0">
 <segment>
-<pinref part="O" gate="G$1" pin="OUT"/>
-<pinref part="3PDT" gate="B" pin="2"/>
-<wire x1="40.64" y1="55.88" x2="45.72" y2="55.88" width="0.1524" layer="91"/>
+<pinref part="U$1" gate="G$1" pin="OUT"/>
+<junction x="12.7" y="43.18"/>
+<label x="15.24" y="43.18" size="1.778" layer="95"/>
+</segment>
+<segment>
+<pinref part="3PDT" gate="A" pin="2"/>
+<junction x="45.72" y="68.58"/>
+<label x="45.72" y="68.58" size="1.778" layer="95" rot="R180"/>
 </segment>
 </net>
-<net name="N$3" class="0">
+<net name="CO" class="0">
+<segment>
+<pinref part="U$1" gate="G$1" pin="CO"/>
+<junction x="12.7" y="40.64"/>
+<label x="15.24" y="40.64" size="1.778" layer="95"/>
+</segment>
+<segment>
+<pinref part="3PDT" gate="A" pin="1"/>
+<junction x="55.88" y="71.12"/>
+<label x="55.88" y="71.12" size="1.778" layer="95"/>
+</segment>
+</net>
+<net name="CI" class="0">
+<segment>
+<pinref part="U$1" gate="G$1" pin="CI"/>
+<junction x="12.7" y="33.02"/>
+<label x="15.24" y="33.02" size="1.778" layer="95"/>
+</segment>
 <segment>
 <pinref part="3PDT" gate="B" pin="1"/>
-<pinref part="CO" gate="G$1" pin="P$1"/>
-<wire x1="55.88" y1="58.42" x2="60.96" y2="58.42" width="0.1524" layer="91"/>
+<junction x="55.88" y="58.42"/>
+<label x="55.88" y="58.42" size="1.778" layer="95"/>
 </segment>
 </net>
-<net name="N$4" class="0">
-<segment>
-<pinref part="3PDT" gate="A" pin="1"/>
-<pinref part="CI" gate="G$1" pin="P$1"/>
-<wire x1="55.88" y1="71.12" x2="60.96" y2="71.12" width="0.1524" layer="91"/>
-</segment>
-</net>
