File: Groupie/Groupie.sch (EAGLE design)
At the start: 10 parts, among them SW1 3PDT

Commit message: Added boards
Parts:
- removed CLR: 4.6k, resistors:RESISTORS.3B
- removed GND1: GND_PADROUND, supply pins:GND_PADROUND
- removed IN, OUT: THONKICONNNEW, MusicThingModular:THONKICONNNEW
- removed LED: LED3MM, diodes:LED3MM
- removed PCB1: EURORACK_PCB12HP, EurorackModularParts:EURORACK_PCB12HP
- removed SW1: 3PDT, switches:3PDT
- removed V1: +9V_PAD, supply pins:+9V_PAD
- added GROUP_VOL: (no value), MusicThingModular:9MM_SNAP-IN_POT_
- added HEADERS: HEADERS8, my_headers:HEADERS8
- added IN_JACK, OUT_JACK: THONKICONNNEW, MusicThingModular:THONKICONNNEW
- added PWR: PJ-037A, Power Socket PJ-037A:PJ-037A
Connections:
- removed net N$1: SW1A.3, SW1B.3
- removed net N$2: LED.C, SW1C.1
- removed net N$3: CLR.1, LED.A
- removed net N$4: CHAIN_IN.TIP, SW1A.1
- removed net N$5: CHAIN_OUT.TIP, SW1B.1
- removed net N$6: IN.TIP, SW1A.2
- removed net N$7: OUT.TIP, SW1B.2
- new net CI: CHAIN_IN.TIP, HEADERS.CI
- new net CO: GROUP_VOL.S, HEADERS.CO
- new net IN: HEADERS.IN, IN_JACK.TIP
- new net N$8: CHAIN_OUT.TIP, GROUP_VOL.E
- new net OUT: HEADERS.OUT, OUT_JACK.TIP
- net +9V: now also HEADERS.+9V, PWR.1; no longer CLR.2, V1.+9V
- net GND: now also CHAIN_IN.SWITCH, CHAIN_OUT.SWITCH, GROUP_VOL.A, HEADERS.G1, HEADERS.G2, HEADERS.GND, IN_JACK.SLEEVE, IN_JACK.SWITCH, OUT_JACK.SLEEVE, OUT_JACK.SWITCH, PWR.2; no longer IN.SLEEVE, OUT.SLEEVE, SW1C.2, SW1C.3
Other:
- moved on the sheet: CHAIN_IN, CHAIN_OUT
