File: Randys_Gut/Randys_Gut.sch (EAGLE design)
At the start: 31 parts, among them Q1 2N1711, Q2 2N1711

Commit message: Added gitignore
Parts:
- removed GI, GO: GND_PADROUND, supply pins:GND_PADROUND
- added U$2: HEADERS6, my_headers:HEADERS6
- BIAS: value B5k -> B5K; device potentiometers:16MM -> MusicThingModular:9MM_SNAP-IN_POT_
- C1: value 47uF -> 100p; device caps-elec:0631 -> caps-film:CAP.2
- C10: value 6.8n -> 100uF; device caps-film:CAP.2 -> caps-elec:0631
- C2: value 4.7uF -> 22uF
- C3: value 470p -> 22uF; device caps-film:CAP.2 -> caps-elec:0501
- C5: value 100p -> 6.8n
- C6: value 100uF -> 6.8n; device caps-elec:0631 -> caps-film:CAP.2
- C7: value 22uF -> 470p; device caps-elec:0501 -> caps-film:CAP.2
- C8: value 22uF -> 4.7uF
- C9: value 6.8n -> 47uF; device caps-film:CAP.2 -> caps-elec:0631
- GREESE: device potentiometers:16MM -> MusicThingModular:9MM_SNAP-IN_POT_
- IN: value IN -> THONKICONNNEW; device supply pins:IN -> MusicThingModular:THONKICONNNEW
- LEVEL: value A100k -> A100K; device potentiometers:16MM -> MusicThingModular:9MM_SNAP-IN_POT_
- OUT: value OUT -> THONKICONNNEW; device supply pins:OUT -> MusicThingModular:THONKICONNNEW
- PWR: value BATTERYBAT2 -> PJ-037A; device jacks:BATTERYBAT2 -> Power Socket PJ-037A:PJ-037A
- R1: value 3.3k -> 1M; device resistors_values:RESISTORS.3B -> resistors:RESISTORS.3B
- R2: value 1k -> 4.7k; device resistors_values:RESISTORS.3B -> resistors:RESISTORS.3B
- R3, R8: value 22k -> 1k
- R4: value 100k -> 68k
- R5: value 4.7k -> 22k
- R6: value 1M -> 22k; device resistors_values:RESISTORS.3B -> resistors:RESISTORS.3B
- R7: value 68k -> 100k
- R9: value 1k -> 3.3k
- TONE: value B50k -> B50K; device potentiometers:16MM -> MusicThingModular:9MM_SNAP-IN_POT_
Connections:
- removed net N$14: LEVEL.3, TONE.2
- new net CI: C1.1, GREESE.E, R1.2, U$2.CI
- new net CO: LEVEL.S, U$2.CO
- new net N$13: LEVEL.E, TONE.S
- net +9V: now also C10.+, PWR.1, R6.2, R9.2, U$2.+9V; no longer C6.+, PWR.P$1, R1.2, R3.2
- net C3: now also C7.2, C8.-, Q2.B, R7.2; no longer C2.-, C3.2, Q1.B, R4.2
- net GND: now also C1.2, C10.-, C3.-, C6.2, C9.-, IN.SLEEVE, IN.SWITCH, LEVEL.A, OUT.SLEEVE, OUT.SWITCH, PWR.2, R1.1, R3.1, R4.2, R8.1, U$2.GND; no longer C1.-, C10.2, C5.2, C6.-, C8.-, GI.GND, GO.GND, LEVEL.1, PWR.P$2, R5.1, R6.1, R7.2, R9.1
- net IN: now also IN.TIP, U$2.IN; no longer C5.1, GREESE.3, IN.IN, R6.2
- net N$1: now also GREESE.A, R2.2; no longer GREESE.1, R5.2
- net N$10: now also BIAS.A, BIAS.S, R9.1; no longer BIAS.1, BIAS.2, R1.1
- net N$11: now also C5.2, R4.1, TONE.E; no longer C9.2, R7.1, TONE.3
- net N$12: now also C6.1, R5.1, TONE.A; no longer C10.1, R8.1, TONE.1
- net N$3: now also C8.+, GREESE.S; no longer C2.+, GREESE.2
- net N$5: now also C9.+, Q1.E, R7.1, R8.2; no longer C1.+, Q2.E, R2.2, R4.1
- net N$6: now also C7.1, Q1.B, Q2.C, R6.1; no longer C3.1, Q1.C, Q2.B, R3.1
- net N$7: now also C3.+, Q2.E, R3.2; no longer C8.+, Q1.E, R9.2
- net N$8: now also BIAS.E, C2.+, Q1.C; no longer BIAS.3, C7.+, Q2.C
- net N$9: now also C2.-, C5.1, R5.2; no longer C7.-, C9.1, R8.2
- net OUT: now also OUT.TIP, U$2.OUT; no longer LEVEL.2, OUT.OUT
Other:
- moved on the sheet: C2, C5, C8, Q1, Q2, R1, R2, R3, R4, R5, R6, R7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
